Commit message: Update pepper_legs.xacro

File: pepper_description/urdf/pepper1.0_generated_urdf/pepper_legs.xacro (robot description, xacro)
@@ -55,3 +55,9 @@
 	</joint>
 	<link name="base_footprint"/>
+	<joint name="base_scan_joint" type="fixed">
+		<parent link="base_footprint"/>
+		<child link="base_scan"/>
+		<origin rpy="0 0 0" xyz="3.14 0 1.57"/>
+	</joint>
+	<link name="base_scan"/>
 </robot>

Commit message: Revert "Update pepper_legs.xacro"
This reverts commit fdc50f9b223846b4aa4a3912a11ce35d3b14adf3.

File: pepper_description/urdf/pepper1.0_generated_urdf/pepper_legs.xacro (robot description, xacro)
@@ -55,9 +55,3 @@
 	</joint>
 	<link name="base_footprint"/>
-	<joint name="base_scan_joint" type="fixed">
-		<parent link="base_footprint"/>
-		<child link="base_scan"/>
-		<origin rpy="0 0 0" xyz="3.14 0 1.57"/>
-	</joint>
-	<link name="base_scan"/>
 </robot>
